Commit message: init

File: legged_gym/resources/robots/h1/urdf/h1.urdf (robot description, URDF)
Before this commit: robot h1_description, 25 links, 24 joints
Links:
- removed link d435_left_imager_link
- removed link d435_rgb_module_link
- removed link imu_link
- removed link logo_link
- removed link mid360_link
- link left_elbow_link: geometry collision cylinder length=0.09 radius=0.03; visual mesh filename=../meshes/left_elbow_link_ball_hand.STL
- link right_elbow_link: geometry collision cylinder length=0.09 radius=0.03; visual mesh filename=../meshes/right_elbow_link_ball_hand.STL
Joints:
- removed joint d435_left_imager_joint
- removed joint d435_rgb_module_joint
- removed joint imu_joint
- removed joint logo_joint
- removed joint mid360_joint
